File: CC2420_module.sch (KiCad schematic (older format))
At the start: 1 part

Commit message: Done
Parts:
- added BQ1: 16MHz Crystal resonator ±20ppm 12pF 80Ω, QFN_DFN:3.2x2.5_QUARTZ, symbol Quartz:X3225_Osc
- added C1, C2: Chip cap. 27 pF NPO 50В 5% 0805, CAPACITOR:CAP_0805, symbol Capacitors:CAPACITOR
- added C10, C9: Chip cap. 0,5 pF NPO 50В 0,25% 0603, CAPACITOR:CAP_0603, symbol Capacitors:CAPACITOR
- added C11, C12: Chip cap. 5,6 pF NPO 50В 0,25% 0805, CAPACITOR:CAP_0805, symbol Capacitors:CAPACITOR
- added C3, C4, C5, C6, C7: Chip cap. 0.1 uF X7R 50В 5% 0805, CAPACITOR:CAP_0805, symbol Capacitors:CAPACITOR
- added C8: Chip cap. 10 uF X5R 16В 10% 0805, CAPACITOR:CAP_0805, symbol Capacitors:CAPACITOR
- added KT1, KT2: KontM3, Connectors:KontaktPl_0,7x2mm, symbol Other:KontM3
- added L1, L2: 0.0075 uH 0805 5%, RESISTORS:RES_0805, symbol Transformers:CDRH6D38NP
- added L3: 0.0056 uH 0805 5%, RESISTORS:RES_0805, symbol Transformers:CDRH6D38NP
- added R1, R2, R3, R4, R5: Chip resistor 0,125W 10kOhm 1% 0805, RESISTORS:RES_0805, symbol Resistors:RES_0805
- added R6: Chip resistor 0,125W 43kOhm 1% 0805, RESISTORS:RES_0805, symbol Resistors:RES_0805
- added XP1: PLD-12, Connectors:PLD-12, symbol Connectors:12contactsXP
- added XS1: KH-SMA-KE-Z, Connectors:KH-SMA-KE-Z, symbol Connectors:5-1814832-1
- DA1: renamed from DA?; LCSC part (none) -> C179669
Connections:
- net labels added: 1V8, 3V3, ATEST1, ATEST2, CCS, CS, EXTRST, FIFO, FIFOP, GND, MISO, MOSI, SCLK, SFD, VREG_EN
- wire segments 0 -> 176
Other:
- moved on the sheet: DA1
